Commit message: robotiq gripper v1.0

File: src/vgn/utils/pal_robotiq_85_gripper.urdf (robot description, URDF)
Before this commit: robot robotiq_85, 15 links, 14 joints
Links:
- removed link gripper_grasping_frame
- removed link gripper_grasping_frame_Y
- removed link gripper_grasping_frame_Z
Joints:
- removed joint gripper_grasping_frame_Y_joint
- removed joint gripper_grasping_frame_Z_joint
- removed joint gripper_grasping_frame_joint
- joint gripper_finger_joint: limit lower=0 upper=0.8 effort=1000.0 velocity=2 -> lower=0 upper=0.8 effort=100.000 velocity=2
- joint gripper_left_inner_finger_joint: limit lower=-0.8757 upper=0 effort=1000.0 velocity=2 -> lower=-0.8757 upper=0 effort=100.000 velocity=2
- joint gripper_left_inner_knuckle_joint: limit lower=0 upper=0.8757 effort=1000.0 velocity=2 -> lower=0 upper=0.8757 effort=100.000 velocity=2
- joint gripper_right_inner_finger_joint: limit lower=-0.8757 upper=0 effort=1000.0 velocity=2 -> lower=-0.8757 upper=0 effort=100.000 velocity=2
- joint gripper_right_inner_knuckle_joint: limit lower=0 upper=0.8757 effort=1000.0 velocity=2 -> lower=0 upper=0.8757 effort=100.000 velocity=2
- joint gripper_right_outer_knuckle_joint: limit lower=0 upper=0.81 effort=1000.0 velocity=2 -> lower=0 upper=0.81 effort=100.000 velocity=2
